Commit message: changed to camera with 78 deg fov and updated quadrotor mesh file to avoid view of landing gear in image

File: agents/quadcopter/quadcopter.urdf.xacro (robot description, xacro)
@@ -8,5 +8,5 @@
   <xacro:property name="namespace" value="quadcopter" />
   <xacro:property name="use_mesh_file" value="true" />
-  <xacro:property name="mesh_file" value="model://quadrotor/meshes/quadrotor_base.dae" />
+  <xacro:property name="mesh_file" value="$(find magicc_sim)/meshes/firefly.dae" />
   <xacro:property name="mass" value="2.856" />
   <xacro:property name="body_width" value="0.505" />
@@ -77,5 +77,5 @@
   <xacro:gps_plugin_macro namespace="${namespace}" parent_link="${namespace}/base_link"/>
   <!-- Fixed Camera -->
-  <xacro:include filename="$(find ibvs_sim)/plugins/xacro/chameleon3_cam.xacro"/>
+  <xacro:include filename="$(find ibvs_sim)/plugins/xacro/chameleon3_3_6mm.xacro"/>
   <xacro:simple_camera
     namespace="${namespace}"

Commit message: getting it all working with the wind

File: agents/quadcopter/quadcopter.urdf.xacro (robot description, xacro)
@@ -11,5 +11,5 @@
   <xacro:property name="mass" value="2.856" />
   <xacro:property name="body_width" value="0.505" />
-  <xacro:property name="body_height" value="0.1" />
+  <xacro:property name="body_height" value="0.001" />
   <xacro:property name="body_inertia">
     <inertia ixx="0.07" ixy="0.0" ixz="0.0" iyy="0.08" iyz="0.0" izz="0.12" />

Commit message: added square root option for ibvs distance and make the copter less wide

File: agents/quadcopter/quadcopter.urdf.xacro (robot description, xacro)
@@ -10,5 +10,5 @@
   <xacro:property name="mesh_file" value="$(find magicc_sim)/meshes/firefly.dae" />
   <xacro:property name="mass" value="2.856" />
-  <xacro:property name="body_width" value="0.505" />
+  <xacro:property name="body_width" value="0.28" />
   <xacro:property name="body_height" value="0.001" />
   <xacro:property name="body_inertia">
